File: hardware/IFB-40003-R02 - I2C_Buttons.brd (EAGLE design)
At the start: 33 x 33 mm, 32 parts, among them J10 CUT_JUMPER_2X, J3 CUTTABLE_JUMPER, J4 POGO_PAD, J5 POGO_PAD, J6 POGO_PAD, J7 POGO_PAD, J8 POGO_PAD, J9 POGO_PAD, SW1 PTS6455MM, SW2 PTS6455MM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

Commit message: updated hardware files
Parts:
- removed J2: (no value), SparkFun-Connectors:1X04_1MM_RA
- removed J3: CUTTABLE_JUMPER, PlayingWithFusion_Breakout-Lib:SMT_CUTTABLE_JUMPER
- added J11, J12: QWIICSIDE, PlayingWithFusion_JST:SM04B-SRSS-TB
- added R9: 100k, rcl:R0603
- J1: value (none) -> CUT_JUMPER_2X; device SparkFun-Connectors:1X04_1MM_RA -> PlayingWithFusion_Breakout-Lib:SMT_2X_CUTTABLE_JUMPER
- moved R8 11.2 mm to (22.9, 22.5), turned to 180 degrees
- moved J10 8.11 mm to (21.0, 12.0), flipped to the top
- moved R4 6.15 mm to (18.2, 22.5), turned to 0 degrees
- moved C1 5.96 mm to (10.5, 23.1), turned to 0 degrees
- moved J1 4.63 mm to (23.4, 18.6), turned to 0 degrees
- moved C2 1.91 mm to (4.88, 20.8), turned to 180 degrees
- moved R5 1.38 mm to (14.9, 22.5), turned to 0 degrees
- moved R6 0.10 mm to (23.9, 15.0)
Connections:
- removed net N$1: J3.2, R8.1, U2.3
- new net ADDR0: J1.1, R8.1, U2.3
- new net ADDR1: J1.3, R9.1, U2.2
- net GND: now also J1.2, J11.1, J12.1; no longer J1.1, J2.1, J3.1
- net SCL: now also J11.4, J12.4; no longer J1.4, J2.4
- net SDA: now also J11.3, J12.3; no longer J1.3, J2.3
- net VCC: now also J11.2, J12.2, R9.2; no longer J1.2, J2.2
Routing:
- net N$1: track 18.2 -> 0.00 mm, vias 2 -> 0
- net ADDR0: track 0.00 -> 16.3 mm
- net ADDR1: track 0.00 -> 15.8 mm
- net VCC: track 77.7 -> 69.8 mm, vias 3 -> 5
- net N$6: track 9.14 -> 2.23 mm, vias 1 -> 0
- net N$3: track 24.4 -> 17.7 mm
- net N$4: track 15.0 -> 19.3 mm
- net N$7: track 6.96 -> 5.17 mm, vias 1 -> 0
- net GND: track 48.0 -> 46.9 mm, vias 28 -> 29
Other:
- board text added: "0 1"
- board text added: "IFB-40003-R01 5x I2C Button Brd"
- board text added: "R9"
- board text removed: "IFB-40003-R01 Quad I2C Buttons"
